File: StepperBoard_Logic/StepperBoard_Logic.kicad_sch (KiCad schematic)
At the start: 84 parts, among them IC1 MP9942GJ-Z, J1 Screw_Terminal_01x02, J10 Conn_02x05_Odd_Even, J2 Conn_01x04, J3 Conn_01x03_MountingPin, J4 Conn_01x06, J5 Conn_01x05, J6 Conn_02x06, J7 Conn_01x05, J8 Conn_01x05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

Commit message: Updated version on GitHub
Parts:
- removed H7, H8: MountingHole, MountingHole:MountingHole_3.2mm_M3, symbol Mechanical:MountingHole
- removed J6: Conn_02x06, Connector_PinHeader_1.27mm:PinHeader_2x06_P1.27mm_Vertical_SMD, symbol Connector_Generic:Conn_02x06_Counter_Clockwise
- C24: value 100n -> 10n
Connections:
- net +24V: no longer J10.2 (Pin_2), J9.2 (Pin_2)
- net +3.3V: now also J10.2 (Pin_2), J9.2 (Pin_2)
- net +3V3: now also L2.2
- net at L2.1, U2.13 (VDDA): now also C17.1, C18.1
Other:
- note added: "Da rivedere"
- note added: "Togliere il doppio pin per il can"
- note removed: "Power mezzanine"
- moved on the sheet: C17, C18, L2
