File: StepperBoard_Power/StepperBoard_Power.kicad_sch (KiCad schematic)
At the start: 65 parts, among them IC1 A4989SLDTR-T, J10 Conn_02x05_Odd_Even, J4 Screw_Terminal_01x04, J6 Conn_02x06, J9 Conn_02x05_Odd_Even, Q1 DMNH10H028SK3Q-13, Q2 DMNH10H028SK3Q-13, Q3 DMNH10H028SK3Q-13, Q4 DMNH10H028SK3Q-13, Q5 DMNH10H028SK3Q-13, Q6 DMNH10H028SK3Q-13, Q7 DMNH10H028SK3Q-13, Q8 DMNH10H028SK3Q-13, SW1 SW_DIP_x02, SW2 SW_DIP_x02

Commit message: Updated version on GitHub
Parts:
- removed C20 (x3): 100u, Capacitor_SMD:C_0402_1005Metric, symbol Device:C
- removed J6: Conn_02x06, Connector_PinHeader_1.27mm:PinHeader_2x06_P1.27mm_Vertical_SMD, symbol Connector_Generic:Conn_02x06_Odd_Even
- removed JP1, JP2, JP3, JP4: SolderJumper_2_Open, Jumper:SolderJumper-2_P1.3mm_Open_RoundedPad1.0x1.5mm, symbol Jumper:SolderJumper_2_Open
- removed R14: 10k, Resistor_SMD:R_0402_1005Metric, symbol Device:R
- added C14, C15: C, Capacitor_SMD:C_0402_1005Metric, symbol Device:C
- added C20 (x3): 68u @ 50V, Capacitor_SMD:CP_Elec_6.3x7.7, symbol Device:C
- added D1: LED, LED_SMD:LED_0201_0603Metric, symbol Device:LED
- added F1: Fuse, Fuse:Fuse_BelFuse_0ZRE0012FF_L8.3mm_W3.8mm, symbol Device:Fuse
- added IC2: VN7007ALHTR, CustomFootprint:OCTAPAK, symbol CustomLibrary:VN7007ALHTR
- added IC3: MCS1802GS-20-Z, CustomFootprint:SOIC127P600X175-8N, symbol CustomLibrary:MCS1802GS-20-Z
- added J1: Screw_Terminal_01x02, TerminalBlock_Phoenix:TerminalBlock_Phoenix_PT-1,5-2-3.5-H_1x02_P3.50mm_Horizontal, symbol Connector:Screw_Terminal_01x02
- added JP1, JP2, JP3, JP4: SolderJumper_3_Bridged12, Jumper:SolderJumper-3_P1.3mm_Bridged2Bar12_RoundedPad1.0x1.5mm_NumberLabels, symbol Jumper:SolderJumper_3_Bridged12
- added R13: 10k, Resistor_SMD:R_0402_1005Metric, symbol Device:R
- added R29: 15k, Resistor_SMD:R_0402_1005Metric, symbol Device:R
- added R6: 3.3k, Resistor_SMD:R_0402_1005Metric, symbol Device:R
- Q1, Q2, Q3, Q4, Q5, Q6, Q7, Q8: footprint Package_TO_SOT_SMD:TO-252-3_TabPin2 -> CustomFootprint:TO-252-2 Tab1
- R25: renamed from R24; value 2k2 -> 3k3
- RV1: value 20k -> 30k
- R_SENSE1: renamed from R9; value 0.03 -> 0.05; footprint Resistor_SMD:R_0402_1005Metric -> Resistor_SMD:R_0612_1632Metric
- R_SENSE2: renamed from R22; value 0.03 -> 0.05; footprint Resistor_SMD:R_0402_1005Metric -> Resistor_SMD:R_0612_1632Metric
- SW1, SW2: footprint Button_Switch_SMD:SW_DIP_SPSTx02_Slide_6.7x6.64mm_W8.61mm_P2.54mm_LowProfile -> Button_Switch_SMD:SW_DIP_SPSTx02_Slide_Copal_CHS-02A_W5.08mm_P1.27mm_JPin
- renumbered C13 to C12, C4 to C5, C5 to C6, C6 to C7, R13 to R14, R25 to R23, R23 to R24, R7 to R8, R8 to R9
Connections:
- net W1_1 is gone; now on net Bridge1_CB: J4.3 (Pin_3)
- net W1_2 is gone; now on net Bridge1_CA: J4.4 (Pin_4)
- net W2_1 is gone; now on net Bridge2_CB: J4.1 (Pin_1)
- net W2_2 is gone; now on net Bridge2_CA: J4.2 (Pin_2)
- net +24V: now also C20.1, D1.2 (A), F1.2, IC2.8 (VCC); no longer J10.2 (Pin_2), J9.2 (Pin_2), Q1.1 (D), Q2.1 (D), Q5.1 (D), Q6.1 (D)
- net +3.3V: now also J10.2 (Pin_2), J9.2 (Pin_2), C14.1, IC3.8 (VCC), R13.1
- net GND: now also C14.2, C15.2, C20.2, C20.2, C20.2, IC2.7 (GND), IC3.5 (GND), J1.2 (Pin_2), R6.2; no longer J9.7 (Pin_7), J9.8 (Pin_8)
- net MS1: now also JP1.2 (C); no longer J10.6 (Pin_6)
- net MS2: now also JP2.2 (C); no longer J10.4 (Pin_4)
- net PFD1: now also JP3.2 (C); no longer J10.3 (Pin_3)
- net PFD2: now also JP4.2 (C); no longer J10.5 (Pin_5)
- net at R12.2, SW1.4: now also JP1.1 (A)
- net at R14.2, SW1.3: now also JP2.1 (A)
- net at R15.2, SW2.3: now also JP4.1 (A)
- net at SW2.4: now also JP3.1 (A), R13.2
- new net: C15.1, IC3.6 (FILT)
- new net: IC2.4 (INPUT), R29.2
- new net: D1.1 (K), R6.1
- new net +24V_Switch: IC2.1 (OUTPUT_1), IC2.2 (OUTPUT_2), IC2.3 (OUTPUT_3), IC3.1 (IP+_1), IC3.2 (IP+_2)
- new net MS1_uC: J10.6 (Pin_6), JP1.3 (B)
- new net MS2_uC: J10.4 (Pin_4), JP2.3 (B)
- new net PFD1_uC: J10.3 (Pin_3), JP3.3 (B)
- new net PFD2_uC: J10.5 (Pin_5), JP4.3 (B)
- new net Sense_uC: IC3.7 (VOUT), J9.8 (Pin_8)
- new net Switch_uC: J9.7 (Pin_7), R29.1
- new net VCC: F1.1, J1.1 (Pin_1)
- new net VDDF: C20.1, C20.1, IC3.3 (IP-_1), IC3.4 (IP-_2), Q1.1 (D), Q2.1 (D), Q5.1 (D), Q6.1 (D)
- no-connect marks 3 -> 5
Other:
- note added: "Current sensor & Switch"
- note added: "Driver"
- note removed: "Power mezzanine"
- moved on the sheet: C12, C20, C6, C7, H1, H2, H3, H4, IC1, J4, Q1, Q2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

Commit message: Added NetTies and NetClasses
Added the NetTies library in CommonComponents folder and defined some NetClasses.
Also fixed the position of some components.
Parts:
- added C20: 10n, Capacitor_SMD:C_0402_1005Metric, symbol Device:C
- added NT1: NetTie_2, NetTies:NetTie-2_SMD_Pad0.2mm, symbol NetTies:NetTie_2
- added NT2: NetTie_2, NetTies:NetTie-2_SMD_Pad0.5mm, symbol NetTies:NetTie_2
- C20: value 100u -> 100n
- J4: footprint TerminalBlock_Phoenix:TerminalBlock_Phoenix_MPT-0,5-4-2.54_1x04_P2.54mm_Horizontal -> TerminalBlock_Phoenix:TerminalBlock_Phoenix_PT-1,5-4-3.5-H_1x04_P3.50mm_Horizontal
Connections:
- net +24V: now also NT1.2; no longer D1.2 (A)
- net +3.3V: now also C20.1
- net GND: now also NT2.2; no longer C12.2, C14.2, C15.2, C20.1, C20.2, IC1.20 (GND), IC2.7 (GND), IC3.5 (GND), J10.10 (Pin_10), J10.7 (Pin_7), J10.8 (Pin_8), J10.9 (Pin_9), J9.10 (Pin_10), J9.9 (Pin_9), R23.2, R25.1, R6.2, SW1.1, SW1.2, SW2.1, SW2.2
- new net: D1.2 (A), NT1.1
- new net GNDD: C12.2, C14.2, C15.2, C20.1, C20.2, C20.2, IC1.20 (GND), IC2.7 (GND), IC3.5 (GND), J10.10 (Pin_10), J10.7 (Pin_7), J10.8 (Pin_8), J10.9 (Pin_9), J9.10 (Pin_10), J9.9 (Pin_9), NT2.1, R23.2, R25.1, R6.2, SW1.1, SW1.2, SW2.1, SW2.2
Other:
- note added: "NetClasses: High Power: high power trace for motor supply (up to 8 Amps) Power: power traces for component supply (up to 1 Amps) LowPower: low power traces (up to 0.5 Amps) PSignal: mixed signal-power traces (up to 1 Amps) HS_Signal: high speed signal (up to 0.5 Amps) LS_Signal: low speed signals (up to 0.5 Amps) Test: very low power test traces (up to 0.1 Amps)"
- moved on the sheet: C14, D1, R25, R29, R6, RV1
